File: SIG60_SOLSHARE/_saved_SIG60_SOLSHARE.sch (KiCad schematic (older format))
At the start: 87 parts, among them J1 CONN_01X02, J2 CONN_02X03, J3 CONN_01X06, J4 CONN_02X03, J7 CONN_02X03, Q1 BSS138, Q2 BSS138, Q3 BSS138, Q4 BSS138, SW1 RESET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

Commit message: Version 0.22 ready for order.
Parts:
- J4: footprint (none) -> Pin_Headers:Pin_Header_Straight_2x03_Pitch2.54mm
Changed lines of the file:
@@
 F 0 "J4" H 2900 4200 50  0000 C CNN
 F 1 "CONN_02X03" H 2900 3800 50  0000 C CNN
-F 2 "" H 2900 2800 50  0001 C CNN
+F 2 "Pin_Headers:Pin_Header_Straight_2x03_Pitch2.54mm" H 2900 2800 50  0001 C CNN
 F 3 "" H 2900 2800 50  0001 C CNN
 	1    2900 4000
